File: arduino/pcb/microswitch.sch (KiCad schematic (older format))
At the start: 10 parts, among them P1 CONN_01X08, P2 CONN_01X02, P3 CONN_01X02, P4 CONN_01X02, P5 CONN_01X02, P6 CONN_01X08

Commit message: Rework enemy animations code. Add dialogs in cutscenes. Finish first custscene and stage
Parts:
- P2, P3, P4, P5: footprint Pin_Headers:Pin_Header_Straight_1x02 -> bornera:mkds_1,5-2
Changed lines of the file:
@@
 F 0 "P2" H 3350 1600 50  0000 C CNN
 F 1 "CONN_01X02" V 3450 1450 50  0000 C CNN
-F 2 "Pin_Headers:Pin_Header_Straight_1x02" H 3350 1450 50  0001 C CNN
+F 2 "bornera:mkds_1,5-2" H 3350 1450 50  0001 C CNN
 F 3 "" H 3350 1450 50  0000 C CNN
 	1    3350 1450
@@
 F 0 "P3" H 3900 1600 50  0000 C CNN
 F 1 "CONN_01X02" V 4000 1450 50  0000 C CNN
-F 2 "Pin_Headers:Pin_Header_Straight_1x02" H 3900 1450 50  0001 C CNN
+F 2 "bornera:mkds_1,5-2" H 3900 1450 50  0001 C CNN
 F 3 "" H 3900 1450 50  0000 C CNN
 	1    3900 1450
@@
 F 0 "P4" H 4450 1600 50  0000 C CNN
 F 1 "CONN_01X02" V 4550 1450 50  0000 C CNN
-F 2 "Pin_Headers:Pin_Header_Straight_1x02" H 4450 1450 50  0001 C CNN
+F 2 "bornera:mkds_1,5-2" H 4450 1450 50  0001 C CNN
 F 3 "" H 4450 1450 50  0000 C CNN
 	1    4450 1450
@@
 F 0 "P5" H 5050 1600 50  0000 C CNN
 F 1 "CONN_01X02" V 5150 1450 50  0000 C CNN
-F 2 "Pin_Headers:Pin_Header_Straight_1x02" H 5050 1450 50  0001 C CNN
+F 2 "bornera:mkds_1,5-2" H 5050 1450 50  0001 C CNN
 F 3 "" H 5050 1450 50  0000 C CNN
 	1    5050 1450
